File: HM10 Breakout.sch (EAGLE design)
At the start: 6 parts, among them U1 HM-10

Commit message: add version & attribution text
Parts:
- added LOGO1: OSHW-LOGOM, Master 2016:OSHW-LOGOM
- C1: value (none) -> 100n
- R1: value (none) -> 1k
Changed lines of the file:
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@@
 <part name="JP2" library="pinhead" library_urn="urn:adsk.eagle:library:325" deviceset="PINHD-1X8" device="" package3d_urn="urn:adsk.eagle:package:22409/2"/>
 <part name="JP3" library="pinhead" library_urn="urn:adsk.eagle:library:325" deviceset="PINHD-1X8" device="" package3d_urn="urn:adsk.eagle:package:22409/2"/>
-<part name="R1" library="rcl" library_urn="urn:adsk.eagle:library:334" deviceset="R-EU_" device="R1206" package3d_urn="urn:adsk.eagle:package:23540/2"/>
-<part name="C1" library="Master 2016" deviceset="C-EU" device="1206"/>
+<part name="R1" library="rcl" library_urn="urn:adsk.eagle:library:334" deviceset="R-EU_" device="R1206" package3d_urn="urn:adsk.eagle:package:23540/2" value="1k"/>
+<part name="C1" library="Master 2016" deviceset="C-EU" device="1206" value="100n"/>
+<part name="LOGO1" library="Master 2016" deviceset="OSHW-LOGO" device="M"/>
 </parts>
 <sheets>
@@
 <attribute name="VALUE" x="90.424" y="18.161" size="1.778" layer="96"/>
 </instance>
+<instance part="LOGO1" gate="G$1" x="88.9" y="96.52" smashed="yes"/>
 </instances>
 <busses>
@@
 </sheet>
 </sheets>
+<errors>
+</errors>
 </schematic>
 </drawing>
