File: HM11 Breakout.brd (EAGLE design)
At the start: 22.9 x 35.6 mm, 7 parts

Commit message: add version & attribution text
Parts:
- added LOGO1: OSHW-LOGOM, Master 2016:OSHW-LOGO-M
- C1: value (none) -> 100n
- R1: value (none) -> 1k
Other:
- board text added: "HM11 Breakout v1.0 Adam Cooper 2023"
Changed lines of the file:
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@@
 <setting verticaltext="up"/>
 </settings>
-<grid distance="0.05" unitdist="inch" unit="inch" style="dots" multiple="1" display="yes" altdistance="0.005" altunitdist="inch" altunit="inch"/>
+<grid distance="0.05" unitdist="inch" unit="inch" style="dots" multiple="1" display="yes" altdistance="0.025" altunitdist="inch" altunit="inch"/>
 <layers>
 <layer number="1" name="Top" color="4" fill="1" visible="yes" active="yes"/>
@@
 <wire x1="6.477" y1="6.985" x2="1.397" y2="6.985" width="0.2032" layer="22"/>
 <wire x1="1.397" y1="6.985" x2="1.27" y2="6.858" width="0.2032" layer="22"/>
+<text x="12.7" y="17.78" size="0.8128" layer="26" font="vector" ratio="15" rot="MR0">HM11 Breakout v1.0
+Adam Cooper 2023</text>
 </plain>
 <attributes>
@@
 <attribute name="NAME" x="13.97" y="4.8895" size="0.4064" layer="25" rot="R90"/>
 </element>
-<element name="R1" library="rcl" library_urn="urn:adsk.eagle:library:334" package="R1206" package3d_urn="urn:adsk.eagle:package:23540/2" value="" x="3.937" y="6.096" smashed="yes" rot="MR180">
+<element name="R1" library="rcl" library_urn="urn:adsk.eagle:library:334" package="R1206" package3d_urn="urn:adsk.eagle:package:23540/2" value="1k" x="3.937" y="6.096" smashed="yes" rot="MR180">
 <attribute name="NAME" x="1.27" y="8.89" size="1.016" layer="26" rot="MR180"/>
 <attribute name="POPULARITY" value="41" x="3.937" y="6.096" size="1.016" layer="28" font="vector" ratio="15" rot="MR180" display="off"/>
@@
 <attribute name="VALUE" x="2.667" y="8.636" size="1.27" layer="28" rot="MR180"/>
 </element>
-<element name="C1" library="Master 2016" package="1206" value="" x="20.066" y="7.874" smashed="yes" rot="MR270">
+<element name="C1" library="Master 2016" package="1206" value="100n" x="20.066" y="7.874" smashed="yes" rot="MR270">
 <attribute name="NAME" x="19.685" y="11.43" size="0.8128" layer="26" font="vector" ratio="10" rot="MR180"/>
 <attribute name="NAME" x="20.066" y="9.779" size="0.8128" layer="34" font="vector" ratio="10" rot="MR270"/>
 <attribute name="VALUE" x="21.971" y="9.779" size="0.8128" layer="28" font="vector" ratio="10" rot="MR270"/>
 </element>
+<element name="LOGO1" library="Master 2016" package="OSHW-LOGO-M" value="OSHW-LOGOM" x="17.145" y="18.415" smashed="yes" rot="MR0"/>
 </elements>
 <signals>
@@
 </drawing>
 <compatibility>
+<note version="6.3" minversion="6.2.2" severity="warning">
+Since Version 6.2.2 text objects can contain more than one line,
+which will not be processed correctly with this version.
+</note>
 <note version="8.2" severity="warning">
 Since Version 8.2, EAGLE supports online libraries. The ids
